Commit message: anything to add?

File: ch6/ch6_ws/src/fishbot_description/urdf/fishbot/fishbot.urdf.xacro (robot description, xacro)
@@ -1,5 +1,6 @@
 <?xml version="1.0"?>
-<!-- Ch 6.2.4, 6.2.5 -->
+<!-- Ch 6.2.4, 6.2.5, 6.4.4 -->
 <robot xmlns:xacro="http://www.ros.org/wiki/xacro" name="fishbot">
+<!-- Include basic components -->
 <xacro:include filename="$(find fishbot_description)/urdf/fishbot/base.urdf.xacro"/>
 <xacro:include filename="$(find fishbot_description)/urdf/fishbot/sensor/camera.urdf.xacro"/>
@@ -8,11 +9,21 @@
 <xacro:include filename="$(find fishbot_description)/urdf/fishbot/actuator/wheel.urdf.xacro"/>
 <xacro:include filename="$(find fishbot_description)/urdf/fishbot/actuator/caster.urdf.xacro"/>
+<!-- Include Gazebo Fortress plugins -->
+<xacro:include filename="$(find fishbot_description)/urdf/fishbot/plugins/gazebo_control_plugins.xacro"/>
+<!-- Robot body -->
 <xacro:base_xacro length="0.12" radius="0.10"/>
+<!-- Sensors -->
 <xacro:camera_xacro xyz="0.10 0.0 0.075"/>
 <xacro:imu_xacro xyz="0.0 0.0 0.02"/>
 <xacro:laser_xacro xyz="0.0 0.0 0.10"/>
+<!-- Actuators -->
 <xacro:wheel_xacro wheel_name="left_wheel" xyz="0.0 0.10 -0.06"/>
 <xacro:wheel_xacro wheel_name="right_wheel" xyz="0.0 -0.10 -0.06"/>
 <xacro:caster_xacro caster_name="front_caster" xyz="0.08 0.0 -0.076"/>
 <xacro:caster_xacro caster_name="back_caster" xyz="-0.08 0.0 -0.076"/>
+<!-- Gazebo Fortress plugins -->
+<!-- <xacro:gazebo_fortress_diff_drive_plugin/>
+<xacro:gazebo_fortress_imu_plugin/>
+<xacro:gazebo_fortress_laser_plugin/>
+<xacro:gazebo_fortress_camera_plugin/> -->
 </robot>

File: ch6/ch6_ws/src/fishbot_description/urdf/fishbot/plugins/gazebo_control_plugins.xacro (robot description, xacro)
@@ -1,7 +1,8 @@
 <?xml version="1.0"?>
 <robot xmlns:xacro="http://www.ros.org/wiki/xacro">
+    <!-- Gazebo Fortress (Ignition Gazebo) compatible differential drive plugin -->
     <xacro:macro name="gazebo_control_plugin">
         <gazebo>
-            <plugin name='diff_drive' filename='libgazebo_ros_diff_drive.so'>
+            <plugin name="gz::sim::systems::DiffDrive" filename="gz-sim-diff-drive-system">
                 <ros>
                     <namespace>/</namespace>
@@ -10,14 +11,14 @@
                 </ros>
                 <update_rate>30</update_rate>
-                <!-- wheels -->
+                <!-- Wheel joints -->
                 <left_joint>left_wheel_joint</left_joint>
                 <right_joint>right_wheel_joint</right_joint>
-                <!-- kinematics -->
+                <!-- Kinematic parameters -->
                 <wheel_separation>0.2</wheel_separation>
                 <wheel_diameter>0.064</wheel_diameter>
-                <!-- limits -->
+                <!-- Limits -->
                 <max_wheel_torque>20</max_wheel_torque>
                 <max_wheel_acceleration>1.0</max_wheel_acceleration>
-                <!-- output -->
+                <!-- Output -->
                 <publish_odom>true</publish_odom>
                 <publish_odom_tf>true</publish_odom_tf>
@@ -27,4 +28,51 @@
             </plugin>
         </gazebo>
-   </xacro:macro>
+    </xacro:macro>
+    <!-- Gazebo Fortress compatible IMU plugin -->
+    <!-- <xacro:macro name="gazebo_fortress_imu_plugin">
+        <gazebo reference="imu_link">
+            <plugin name="gz::sim::systems::Imu" filename="gz-sim-imu-system">
+                <ros>
+                    <namespace>/</namespace>
+                    <remapping>imu:=imu</remapping>
+                </ros>
+                <update_rate>100</update_rate>
+                <topic>imu</topic>
+            </plugin>
+        </gazebo>
+    </xacro:macro> -->
+    <!-- Gazebo Fortress compatible LiDAR plugin -->
+    <!-- <xacro:macro name="gazebo_fortress_laser_plugin">
+        <gazebo reference="laser_link">
+            <plugin name="gz::sim::systems::LaserScan" filename="gz-sim-laserscan-system">
+                <ros>
+                    <namespace>/</namespace>
+                    <remapping>scan:=scan</remapping>
+                </ros>
+                <update_rate>10</update_rate>
+                <topic>scan</topic>
+                <min_angle>-3.14159</min_angle>
+                <max_angle>3.14159</max_angle>
+                <min_range>0.1</min_range>
+                <max_range>10.0</max_range>
+                <range_resolution>0.01</range_resolution>
+            </plugin>
+        </gazebo>
+    </xacro:macro> -->
+    <!-- Gazebo Fortress compatible camera plugin -->
+    <!-- <xacro:macro name="gazebo_fortress_camera_plugin">
+        <gazebo reference="camera_link">
+            <plugin name="gz::sim::systems::Camera" filename="gz-sim-camera-system">
+                <ros>
+                    <namespace>/</namespace>
+                    <remapping>image_raw:=camera/image_raw</remapping>
+                </ros>
+                <update_rate>30</update_rate>
+                <topic>camera/image_raw</topic>
+                <width>640</width>
+                <height>480</height>
+                <format>R8G8B8</format>
+            </plugin>
+        </gazebo>
+    </xacro:macro> -->
 </robot>
