Commit message: debugging laser rays

File: ch6/ch6_ws/src/fishbot_description/urdf/fishbot/base.urdf.xacro (robot description, xacro)
@@ -34,5 +34,5 @@
         </link>
         <link name="base_footprint"/>
-        <joint name="joint_name" type="fixed">
+        <joint name="base_footprint_joint" type="fixed">
             <origin xyz="0.0 0.0 ${length/2.0 + 0.032 - 0.001}" rpy="0.0 0.0 0.0"/>
             <parent link="base_footprint"/>

File: ch6/ch6_ws/src/fishbot_description/urdf/fishbot/fishbot.urdf.xacro (robot description, xacro)
@@ -11,4 +11,5 @@
 <!-- Include Gazebo Fortress plugins -->
 <xacro:include filename="$(find fishbot_description)/urdf/fishbot/plugins/gazebo_control_plugins.xacro"/>
+<xacro:include filename="$(find fishbot_description)/urdf/fishbot/plugins/gazebo_sensor_plugins.xacro"/>
 <!-- Robot body -->
 <xacro:base_xacro length="0.12" radius="0.10"/>
@@ -24,3 +25,4 @@
 <!-- Gazebo Fortress plugins -->
 <xacro:gazebo_control_plugin/>
+<xacro:gazebo_sensor_plugin/>
 </robot>

File: ch6/ch6_ws/src/fishbot_description/urdf/fishbot/plugins/gazebo_control_plugins.xacro (robot description, xacro)
@@ -2,25 +2,19 @@
 <robot xmlns:xacro="http://www.ros.org/wiki/xacro">
   <xacro:macro name="gazebo_control_plugin">
-    <!-- Put plugin under a top-level <gazebo> so URDF->SDF conversion keeps it -->
     <gazebo>
+      <!-- Differential drive -->
       <plugin
         filename="libignition-gazebo-diff-drive-system.so"
         name="ignition::gazebo::systems::DiffDrive">
-        <!-- Wheels (repeat tags if multiple wheels per side) -->
         <left_joint>left_wheel_joint</left_joint>
         <right_joint>right_wheel_joint</right_joint>
-        <!-- Geometry -->
         <wheel_separation>0.2</wheel_separation>
-        <!-- 0.064 diameter -> 0.032 radius -->
         <wheel_radius>0.032</wheel_radius>
-        <!-- Topics on Gazebo Transport (you can keep defaults if you like) -->
         <topic>/model/fishbot/cmd_vel</topic>
         <odom_topic>/model/fishbot/odometry</odom_topic>
         <tf_topic>/model/fishbot/tf</tf_topic>
-        <!-- Frames + publish rate -->
         <frame_id>odom</frame_id>
         <child_frame_id>base_footprint</child_frame_id>
         <odom_publish_frequency>30</odom_publish_frequency>
-        <!-- Optional motion limits (examples) -->
         <max_linear_velocity>1.0</max_linear_velocity>
         <max_angular_velocity>3.0</max_angular_velocity>
@@ -28,4 +22,10 @@
         <max_angular_acceleration>6.0</max_angular_acceleration>
       </plugin>
+      <!-- Publish joint states for ROS -->
+      <plugin
+        filename="libignition-gazebo6-joint-state-publisher-system.so"
+        name="ignition::gazebo::systems::JointStatePublisher">
+        <topic>/model/fishbot/joint_state</topic>
+      </plugin>
     </gazebo>
   </xacro:macro>
