Commit message: lidar, imu, camera working

File: ch6/ch6_ws/src/fishbot_description/urdf/fishbot/plugins/gazebo_sensor_plugins.xacro (robot description, xacro)
@@ -5,5 +5,5 @@
     <!-- LIDAR (2D) -->
     <gazebo reference="laser_link">
-      <sensor name="gpu_lidar" type="gpu_lidar">
+      <sensor name='gpu_lidar' type='gpu_lidar'>
         <!-- Publish rate & topic -->
         <update_rate>10</update_rate>
@@ -17,6 +17,6 @@
               <samples>360</samples>
               <resolution>1</resolution>
-              <min_angle>0</min_angle>
-              <max_angle>6.283185307179586</max_angle> <!-- 2π -->
+              <min_angle>-3.141592653589793</min_angle>
+              <max_angle> 3.141592653589793</max_angle>
             </horizontal>
           </scan>
@@ -26,9 +26,111 @@
             <resolution>0.015</resolution>
           </range>
+          <noise>
+              <type>gaussian</type>
+              <mean>0.0</mean>
+              <stddev>0.01</stddev>
+          </noise>
         </ray>
-        <always_on>true</always_on>
+        <always_on>1</always_on>
         <visualize>true</visualize>
       </sensor>
     </gazebo>
+    <gazebo>
+      <plugin filename="libignition-gazebo-sensors-system.so" name="ignition::gazebo::systems::Sensors">
+          <render_engine>ogre</render_engine>
+      </plugin>
+    </gazebo>
+    <!-- IMU Sensor -->
+    <gazebo reference="imu_link">
+        <sensor name="imu_sensor" type="imu">
+            <update_rate>100</update_rate>
+            <topic>/model/fishbot/imu</topic>
+            <gz_frame_id>imu_link</gz_frame_id>
+            <always_on>true</always_on>
+            <visualize>true</visualize>
+            <plugin filename="gz-sim-imu-system" name="gz::sim::systems::Imu">
+            </plugin>
+            <imu>
+                <angular_velocity>
+                    <x>
+                        <noise type="gaussian">
+                            <mean>0.0</mean>
+                            <stddev>2e-4</stddev>
+                            <bias_mean>0.0000075</bias_mean>
+                            <bias_stddev>0.0000008</bias_stddev>
+                        </noise>
+                    </x>
+                    <y>
+                        <noise type="gaussian">
+                            <mean>0.0</mean>
+                            <stddev>2e-4</stddev>
+                            <bias_mean>0.0000075</bias_mean>
+                            <bias_stddev>0.0000008</bias_stddev>
+                        </noise>
+                    </y>
+                    <z>
+                        <noise type="gaussian">
+                            <mean>0.0</mean>
+                            <stddev>2e-4</stddev>
+                            <bias_mean>0.0000075</bias_mean>
+                            <bias_stddev>0.0000008</bias_stddev>
+                        </noise>
+                    </z>
+                </angular_velocity>
+                <linear_acceleration>
+                    <x>
+                        <noise type="gaussian">
+                            <mean>0.0</mean>
+                            <stddev>1.7e-2</stddev>
+                            <bias_mean>0.1</bias_mean>
+                            <bias_stddev>0.001</bias_stddev>
+                        </noise>
+                    </x>
+                    <y>
+                        <noise type="gaussian">
+                            <mean>0.0</mean>
+                            <stddev>1.7e-2</stddev>
+                            <bias_mean>0.1</bias_mean>
+                            <bias_stddev>0.001</bias_stddev>
+                        </noise>
+                    </y>
+                    <z>
+                        <noise type="gaussian">
+                            <mean>0.0</mean>
+                            <stddev>1.7e-2</stddev>
+                            <bias_mean>0.1</bias_mean>
+                            <bias_stddev>0.001</bias_stddev>
+                        </noise>
+                    </z>
+                </linear_acceleration>
+            </imu>
+        </sensor>
+    </gazebo>
+    <!-- Camera Sensor -->
+    <gazebo reference="camera_link">
+        <sensor name="camera" type="camera">
+            <update_rate>15</update_rate>
+            <topic>/model/fishbot/camera/image_raw</topic>
+            <gz_frame_id>camera_optical_link</gz_frame_id>
+            <always_on>true</always_on>
+            <visualize>true</visualize>
+            <camera>
+                <horizontal_fov>1.5009831567</horizontal_fov>
+                <image>
+                    <width>800</width>
+                    <height>600</height>
+                    <format>R8G8B8</format>
+                </image>
+                <distortion>
+                    <k1>0.0</k1>
+                    <k2>0.0</k2>
+                    <k3>0.0</k3>
+                    <p1>0.0</p1>
+                    <p2>0.0</p2>
+                    <center>0.5 0.5</center>
+                </distortion>
+            </camera>
+        </sensor>
+    </gazebo>
   </xacro:macro>
 </robot>

File: ch6/ch6_ws/src/fishbot_description/urdf/fishbot/sensor/camera.urdf.xacro (robot description, xacro)
@@ -32,4 +32,5 @@
             <xacro:box_inertia m="0.10" w="0.02" h="0.10" d="0.02"/>
         </link>
+        <link name="camera_optical_link"></link>
         <!-- Joints -->
         <joint name="camera_joint" type="fixed">
@@ -38,4 +39,9 @@
             <origin xyz="${xyz}" rpy="0.0 0.0 0.0"/>
         </joint>
+        <joint name="camera_optical_joint" type="fixed">
+            <parent link="camera_link"/>
+            <child link="camera_optical_link"/>
+            <origin xyz="0.0 0.0 0.0" rpy="${-pi/2.0} 0.0 ${-pi/2.0}"/>
+        </joint>
     </xacro:macro>
 </robot>
